File: hardware/mp3_player.kicad_sch (KiCad schematic)
At the start: 0 parts

Commit message: hardware design
Parts:
- added C1, C12, C14, C16, C18, C2, C20, C22, C3, C4, C5, C6, C8: 0.1uF, symbol Device:C
- added C10, C11: 2.2uF, symbol Device:C
- added C13, C15, C17, C19, C21, C23, C9: 10uF, symbol Device:C_Polarized
- added C7: 100uF, symbol Device:C_Polarized
- added J1: AudioJack3, symbol Connector_Audio:AudioJack3
- added J2: Micro_SD_Card_Det1, symbol Connector:Micro_SD_Card_Det1
- added Q1: 2N7002, Package_TO_SOT_SMD:SOT-23, symbol Transistor_FET:2N7002
- added Q2: BSS84, Package_TO_SOT_SMD:SOT-23, symbol Transistor_FET:BSS84
- added R1, R2, R5, R7, R8: 1K, symbol Device:R
- added R10, R11, R12, R13, R14, R3, R4, R6, R9: 10K, symbol Device:R
- added R15, R16: 470R, symbol Device:R
- added R17, R18, R19: 22R, symbol Device:R
- added SW1: RotaryEncoder_Switch, symbol Device:RotaryEncoder_Switch
- added SW2, SW3: SW_Push, symbol Switch:SW_Push
- added U1: ESP32-S3-WROOM-1, RF_Module:ESP32-S3-WROOM-1, symbol RF_Module:ESP32-S3-WROOM-1
- added U2: PCM5100A, Package_SO:TSSOP-20_4.4x6.5mm_P0.65mm, symbol Audio:PCM5100A
- added U3: TPA6110A2DGN, Package_SO:HVSSOP-8-1EP_3x3mm_P0.65mm_EP1.57x1.89mm, symbol Amplifier_Audio:TPA6110A2DGN
- added U4: ST7735S LCD, symbol other_modules:ST7735S_128x160_LCD
- added U5: 74HC14, symbol 74xx:74HC14
Connections:
- new net: J2.1 (DAT2), R12.1
- new net: R19.2, U2.13 (BCK)
- new net: C10.1, U2.2 (CAPP)
- new net: C10.2, U2.4 (CAPM)
- new net: R10.1, R8.1, SW1.A
- new net: R7.1, R9.1, SW1.B
- new net: R5.2, R6.1, SW1.S2
- new net: R16.1, U2.7 (OUTR)
- new net: C11.1, U2.5 (VNEG)
- new net: J2.8 (DAT1), R11.1
- new net: C3.1, R5.1, U5.5
- new net: Q1.3 (D), Q2.2 (S), U3.3 (SHDN)
- new net: C1.1, R1.2, U5.1
- new net: R15.1, U2.6 (OUTL)
- new net: R2.1, R4.1, SW2.1
- new net: C18.1, C19.1, U2.18 (LDOO)
- new net: R1.1, R3.1, SW3.1
- new net: R18.2, U2.14 (DIN)
- new net: R17.2, U2.15 (LRCK)
- new net: C4.1, R7.2, U5.11
- new net: C2.1, R2.2, U5.3
- new net: C5.1, R8.2, U5.9
- new net +3V3: C22.1, C23.1, C6.1, C7.1, C8.1, C9.1, J2.4 (VDD), R10.2, R11.2, R12.2, R13.2, R14.2, R3.2, R4.2, R6.2, R9.2, U1.2 (3V3), U4. (VDD), U5.14 (VCC)
- new net +3V3_A: C12.1, C13.1, C14.1, C15.1, C20.1, C21.1, U2.1 (CPVDD), U2.8 (AVDD), U3.6 (VDD)
- new net +3V3_D: C16.1, C17.1, Q2.3 (D), U2.20 (DVDD)
- new net AGND: C11.2, C12.2, C13.2, C14.2, C15.2, C20.2, C21.2, U2.3 (CPGND), U2.9 (AGND), U3.2 (GND), U3.9 (GND)
- new net BTN1: U1.4 (IO4), U5.4
- new net BTN2: U1.5 (IO5), U5.2
- new net DAC_BCK: R19.1, U1.20 (IO12)
- new net DAC_DIN: R18.1, U1.21 (IO13)
- new net DAC_LRCK: R17.1, U1.22 (IO14)
- new net DAC_MUTE: Q1.1 (G), Q2.1 (G), U2.17 (XSMT)
- new net E_BTN: U1.8 (IO15), U5.6
- new net E_CCW: U1.7 (IO7), U5.8
- new net E_CW: U1.6 (IO6), U5.10
- new net GND: C1.2, C16.2, C17.2, C18.2, C19.2, C2.2, C22.2, C23.2, C3.2, C4.2, C5.2, C6.2, C7.2, C8.2, C9.2, J2.6 (VSS), J2.SH (SHIELD), Q1.2 (S), SW1.C, SW1.S1, SW2.2, SW3.2, U1.1 (GND), U1.40 (GND), U1.41 (GND), U2.10 (DEMP), U2.11 (FLT), U2.12 (SCK), U2.16 (FMT), U2.19 (DGND), U4.1 (GND), U5.13, U5.7 (GND)
- new net GP1: U1.39 (IO1), U4. (VDD)
- new net GP2: U1.38 (IO2), U4. (VDD)
- new net GP21: U1.23 (IO21), U4. (VDD)
- new net GP38: U1.31 (IO38), U4. (VDD)
- new net GP47: U1.24 (IO47), U4. (VDD)
- new net GP48: U1.25 (IO48), U4. (VDD)
- new net OUTL: R15.2, U3.8 (IN1-)
- new net OUTR: R16.2, U3.4 (IN2-)
- new net SD_CARDCS: J2.2 (DAT3/CD), R14.1, U1.12 (IO8)
- new net SD_DET: J2.9 (DET)
- new net SD_MISO: J2.7 (DAT0), U1.19 (IO11)
- new net SD_MOSI: J2.3 (CMD), R13.1, U1.18 (IO10)
- new net SD_SCK: J2.5 (CLK), U1.17 (IO9)
- no-connect marks 0 -> 1
Other:
- note added: "Star all AGND"
